Commit message: Ground ER15 limits in public and engineering data
The planner and control-facing API now derive ER15-1400 joint speed limits from EFORT's public product leaflet. Missing actuator torque limits are filled with documented engineering defaults for method validation and synchronized into the cuRobo URDF effort fields plus the control torque clamp.

Constraint: EFORT public leaflet publishes joint speed and wrist payload torque/inertia, but not J1-J6 actuator torque limits
Constraint: Method validation needs reasonable torque saturation values before controller data is available
Rejected: Keep effort=1 parser sentinel | no longer useful once engineering defaults are allowed
Rejected: Treat wrist payload torque as actuator torque | wrong physical meaning
Confidence: medium
Scope-risk: moderate
Directive: Treat actuator_torque_upper_nm as engineering defaults until drive/controller data replaces them
Tested: pytest -q in IsaacLab Python
Tested: compare_cspace_profiles.py --no-warmup --json in IsaacLab Python
Tested: run_quickmove_demo.sh in IsaacLab Python
Not-tested: Real controller torque saturation behavior

File: assets/er15_1400/ER15-1400-fulldyn-curobo.urdf (robot description, URDF)
Before this commit: robot ER15-1400, 7 links, 6 joints
Joints:
- joint joint_1: limit lower=-2.967 upper=2.967 effort=1000 velocity=4.53785606 -> lower=-2.967 upper=2.967 effort=420.0 velocity=4.53785606
- joint joint_2: limit lower=-2.7925 upper=1.5707963267 effort=1000 velocity=4.45058959 -> lower=-2.7925 upper=1.5707963267 effort=520.0 velocity=4.45058959
- joint joint_3: limit lower=-1.4835 upper=3.0543 effort=1000 velocity=3.66519143 -> lower=-1.4835 upper=3.0543 effort=360.0 velocity=3.66519143
- joint joint_4: limit lower=-3.316 upper=3.316 effort=1000 velocity=7.85398163 -> lower=-3.316 upper=3.316 effort=120.0 velocity=7.85398163
- joint joint_5: limit lower=-2.2689 upper=2.2689 effort=1000 velocity=7.85398163 -> lower=-2.2689 upper=2.2689 effort=100.0 velocity=7.85398163
- joint joint_6: limit lower=-6.2832 upper=6.2832 effort=1000 velocity=10.47197551 -> lower=-6.2832 upper=6.2832 effort=60.0 velocity=10.47197551

Commit message: Add torque-limited retiming for ER15 cycle time
Acceleration and jerk are no longer treated as direct robot hardware limits. The quickmove path is audited with MuJoCo inverse dynamics and uniformly retimed toward the velocity/torque boundary, giving a first torque-limited time-optimal pass on the ER15 example.

Constraint: ER15 actuator torques are engineering defaults until drive/controller data is available
Constraint: MuJoCo J1 static gravity torque must remain near zero because J1 is the vertical base yaw axis
Rejected: Keep acceleration/jerk as direct hard limits | they are not direct robot hardware constraints
Rejected: Use mj_inverse directly for audit | produced inconsistent J1 static torque in this call path
Confidence: medium
Scope-risk: moderate
Directive: Preserve the M(q)qdd + qfrc_bias inverse-dynamics formulation unless a validated dynamics backend replaces it
Tested: pytest -q in IsaacLab Python
Tested: examples/torque_limited_time_scaling.py --no-warmup --json in IsaacLab Python
Tested: run_quickmove_demo.sh in IsaacLab Python
Not-tested: Real ER15 controller torque/current logs

File: assets/er15_1400/ER15-1400-fulldyn-curobo.urdf (robot description, URDF)
Before this commit: robot ER15-1400, 7 links, 6 joints
Joints:
- joint joint_1: limit lower=-2.967 upper=2.967 effort=420.0 velocity=4.53785606 -> lower=-2.967 upper=2.967 effort=1800.0 velocity=4.53785606
- joint joint_2: limit lower=-2.7925 upper=1.5707963267 effort=520.0 velocity=4.45058959 -> lower=-2.7925 upper=1.5707963267 effort=1200.0 velocity=4.45058959
- joint joint_3: limit lower=-1.4835 upper=3.0543 effort=360.0 velocity=3.66519143 -> lower=-1.4835 upper=3.0543 effort=700.0 velocity=3.66519143
- joint joint_4: limit lower=-3.316 upper=3.316 effort=120.0 velocity=7.85398163 -> lower=-3.316 upper=3.316 effort=180.0 velocity=7.85398163
- joint joint_5: limit lower=-2.2689 upper=2.2689 effort=100.0 velocity=7.85398163 -> lower=-2.2689 upper=2.2689 effort=140.0 velocity=7.85398163
- joint joint_6: limit lower=-6.2832 upper=6.2832 effort=60.0 velocity=10.47197551 -> lower=-6.2832 upper=6.2832 effort=90.0 velocity=10.47197551
